File: smol.kicad_pcb (KiCad board)
At the start: 2 copper layers, 164 parts, among them Q1 BSS138, SW1 1U, SW10 1U, SW11 1U, SW12 1U, SW13 1U, SW14 2U, SW15 2U, SW16 1U, SW17 1U, SW18 1U, SW19 1U, SW2 1U, SW20 1U, SW21 1U, SW22 1U, SW23 1U, SW24 1U, SW25 1U, SW26 1U, SW27 1U, SW28 1U, SW29 1U, SW3 1U, SW30 1U, SW31 1U, SW32 1U, SW33 1U, SW34 1U, SW35 1U, SW36 1U, SW37 1U, SW38 1U, SW39 1U, SW4 1U, SW40 1U, SW41 1U, SW42 2U, SW43 2U, SW44 1U, SW45 1U, SW46 1U, SW47 1U, SW48 1U, SW49 1U, SW5 1U, SW50 1U, SW51 1U, SW52 1U, SW53 1U, SW54 1U, SW55 1U, SW56 1U, SW57 1U, SW58 1U, SW59 1U, SW6 1U, SW60 1U, SW61 1U, SW62 1U, SW63 2U, SW64 1U, SW65 1U, SW66 1U, SW67 1U, SW68 1U, SW69 1U, SW7 1U, SW70 1U, SW8 1U, SW9 1U, U1 MiniF4x1Cx_V31

Commit message: add ground plane and adjust decoupling caps
Parts:
- moved C4 7.32 mm to (295.3, 84.9), turned to 180 degrees
- moved C5 7.32 mm to (295.3, 104.0), turned to 180 degrees
- moved C1 7.32 mm to (295.3, 27.8), turned to 180 degrees
- moved C2 7.32 mm to (295.3, 46.8), turned to 180 degrees
- moved C3 7.32 mm to (295.3, 65.9), turned to 180 degrees
- moved C6 7.32 mm to (1.59, 94.5), turned to 0 degrees
- moved C7 7.32 mm to (1.59, 75.4), turned to 0 degrees
- moved C9 7.32 mm to (1.59, 37.3), turned to 0 degrees
- moved C10 7.32 mm to (1.59, 18.3), turned to 0 degrees
- moved C8 7.32 mm to (1.59, 56.4), turned to 0 degrees
Routing:
- added copper zone on F.Cu, net GND

Commit message: last adjustments before routing
Parts:
- moved R2 89.1 mm to (32.5, 3.97)
- moved Q1 88.3 mm to (37.3, 3.97)
- moved R1 81.0 mm to (42.1, 3.97), turned to 90 degrees
- moved U1 22.1 mm to (-0.79, 3.17)

Commit message: route matrix rows
Parts:
- moved D8 3.55 mm to (145.3, 26.2), turned to 270 degrees
- moved D21 3.27 mm to (145.3, 45.2), turned to 270 degrees
- moved D23 3.27 mm to (183.4, 45.2), turned to 270 degrees
- moved D24 3.27 mm to (202.4, 45.2), turned to 270 degrees
- moved D26 3.27 mm to (240.5, 45.2), turned to 270 degrees
- moved D27 3.27 mm to (259.6, 45.2), turned to 270 degrees
- moved D28 3.27 mm to (278.6, 45.2), turned to 270 degrees
- moved D36 3.27 mm to (145.3, 64.3), turned to 270 degrees
- moved D38 3.27 mm to (183.4, 64.3), turned to 270 degrees
- moved D39 3.27 mm to (202.4, 64.3), turned to 270 degrees
- moved D41 3.27 mm to (240.5, 64.3), turned to 270 degrees
- moved D42 3.27 mm to (269.1, 64.3), turned to 270 degrees
- moved D49 3.27 mm to (145.3, 83.3), turned to 270 degrees
- moved D51 3.27 mm to (183.4, 83.3), turned to 270 degrees
- moved D52 3.27 mm to (202.4, 83.3), turned to 270 degrees
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Routing:
- net ROW5: track 0.00 -> 266.7 mm
- net ROW4: track 0.00 -> 257.2 mm
- net ROW3: track 0.00 -> 257.2 mm
- net ROW2: track 0.00 -> 257.2 mm
- net ROW1: track 0.00 -> 257.2 mm
- net Net-(D40-Pad1): track 0.00 -> 5.04 mm
- net Net-(D37-Pad1): track 0.00 -> 5.04 mm
- net Net-(D67-Pad1): track 0.00 -> 5.04 mm
- net Net-(D64-Pad1): track 0.00 -> 5.04 mm
- net Net-(D53-Pad1): track 0.00 -> 5.04 mm
- net Net-(D50-Pad1): track 0.00 -> 5.04 mm
- net Net-(D9-Pad1): track 0.00 -> 5.04 mm
- net Net-(D12-Pad1): track 0.00 -> 5.04 mm
- net Net-(D25-Pad1): track 0.00 -> 5.04 mm
- net Net-(D22-Pad1): track 0.00 -> 5.04 mm
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Other:
- net class Default: clearance 0.2 -> 0.3; trace_width 0.25 -> 0.3; via_drill 0.4 -> 0.5
- rule trace_clearance: 0.2 -> 0.3

Commit message: route matrix columns
Routing:
- net COL4: track 0.00 -> 115.0 mm
- net COL5: track 0.00 -> 115.0 mm
- net COL3: track 0.00 -> 115.0 mm
- net COL2: track 0.00 -> 115.0 mm
- net COL6: track 0.00 -> 115.0 mm
- net COL13: track 0.00 -> 108.6 mm
- net COL7: track 0.00 -> 107.4 mm
- net COL8: track 0.00 -> 103.5 mm
- net COL12: track 0.00 -> 103.5 mm
- net COL10: track 0.00 -> 103.5 mm
- net COL9: track 0.00 -> 103.5 mm
- net COL11: track 0.00 -> 103.5 mm
- net COL1: track 0.00 -> 92.0 mm
- net COL14: track 0.00 -> 88.0 mm

Commit message: route leds
Routing:
- net Net-(RGB5-Pad4): track 0.00 -> 302.2 mm
- net +5V: track 0.00 -> 251.6 mm
- net Net-(RGB8-Pad4): track 0.00 -> 15.5 mm
- net Net-(RGB7-Pad4): track 0.00 -> 15.5 mm
- net Net-(RGB2-Pad4): track 0.00 -> 15.5 mm
- net Net-(RGB10-Pad2): track 0.00 -> 15.5 mm
- net Net-(RGB6-Pad4): track 0.00 -> 15.5 mm
- net Net-(RGB3-Pad4): track 0.00 -> 15.5 mm
- net Net-(RGB1-Pad4): track 0.00 -> 15.5 mm
- net Net-(RGB4-Pad4): track 0.00 -> 15.5 mm
Other:
- net class PWR added: clearance 0.45, trace_width 0.45, via_dia 0.9, via_drill 0.6
Changed lines of the file:
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@@
     (thickness 1.6)
     (drawings 0)
-    (tracks 307)
+    (tracks 392)
     (zones 0)
     (modules 164)
@@
     (uvia_dia 0.3)
     (uvia_drill 0.1)
-    (add_net +3V3)
-    (add_net +5V)
     (add_net COL1)
     (add_net COL10)
@@
     (add_net COL8)
     (add_net COL9)
-    (add_net GND)
     (add_net "Net-(D1-Pad1)")
     (add_net "Net-(D10-Pad1)")
@@
     (add_net ROW5)
   )
+  (net_class PWR ""
+    (clearance 0.45)
+    (trace_width 0.45)
+    (via_dia 0.9)
+    (via_drill 0.6)
+    (uvia_dia 0.3)
+    (uvia_drill 0.1)
+    (add_net +3V3)
+    (add_net +5V)
+    (add_net GND)
+  )
   (module LED_SMD:LED_SK6812_PLCC4_5.0x5.0mm_P3.2mm locked (layer F.Cu)
     (at 0.79375 23.01875 270)
@@
   (segment (start 274.79625 56.03875) (end 274.79625 65.56375) (width 0.3) (layer F.Cu) (net 89))
   (segment (start 284.32125 75.08875) (end 284.32125 94.13875) (width 0.3) (layer F.Cu) (net 89))
+  (segment (start 294.46875 82.61875) (end 294.48125 82.61875) (width 0.3) (layer F.Cu) (net 100))
+  (segment (start 294.46875 101.63125) (end 294.46875 101.66875) (width 0.3) (layer F.Cu) (net 100))
+  (segment (start 294.325 25.6125) (end 294.46875 25.46875) (width 0.3) (layer F.Cu) (net 100))
+  (segment (start 294.325 44.6625) (end 294.46875 44.51875) (width 0.3) (layer F.Cu) (net 100))
+  (segment (start 294.325 63.7125) (end 294.46875 63.56875) (width 0.3) (layer F.Cu) (net 100))
+  (segment (start 294.325 82.7625) (end 294.46875 82.61875) (width 0.3) (layer F.Cu) (net 100))
+  (segment (start 2.39375 96.80625) (end 2.39375 96.76875) (width 0.3) (layer F.Cu) (net 100))
+  (segment (start 2.5375 96.625) (end 2.39375 96.76875) (width 0.3) (layer F.Cu) (net 100))
+  (segment (start 294.325 101.8125) (end 294.46875 101.66875) (width 0.45) (layer F.Cu) (net 100))
+  (segment (start 294.46875 27.6375) (end 294.325 27.78125) (width 0.45) (layer F.Cu) (net 100))
+  (segment (start 294.46875 25.46875) (end 294.46875 27.6375) (width 0.45) (layer F.Cu) (net 100))
+  (segment (start 294.46875 46.6875) (end 294.325 46.83125) (width 0.45) (layer F.Cu) (net 100))
+  (segment (start 294.46875 44.51875) (end 294.46875 46.6875) (width 0.45) (layer F.Cu) (net 100))
+  (segment (start 294.46875 65.7375) (end 294.325 65.88125) (width 0.45) (layer F.Cu) (net 100))
+  (segment (start 294.46875 63.56875) (end 294.46875 65.7375) (width 0.45) (layer F.Cu) (net 100))
+  (segment (start 294.46875 84.7875) (end 294.325 84.93125) (width 0.45) (layer F.Cu) (net 100))
+  (segment (start 294.46875 82.61875) (end 294.46875 84.7875) (width 0.45) (layer F.Cu) (net 100))
+  (segment (start 294.46875 103.8375) (end 294.325 103.98125) (width 0.45) (layer F.Cu) (net 100))
+  (segment (start 294.46875 101.66875) (end 294.46875 103.8375) (width 0.45) (layer F.Cu) (net 100))
+  (segment (start 296.9375 23) (end 294.46875 25.46875) (width 0.45) (layer F.Cu) (net 100))
+  (segment (start 300.7 23) (end 296.9375 23) (width 0.45) (layer F.Cu) (net 100))
+  (segment (start 300.7 99.2) (end 300.7 23) (width 0.45) (layer F.Cu) (net 100))
+  (segment (start 296.9375 99.2) (end 300.7 99.2) (width 0.45) (layer F.Cu) (net 100))
+  (segment (start 294.46875 101.66875) (end 296.9375 99.2) (width 0.45) (layer F.Cu) (net 100))
+  (segment (start 296.8875 42.1) (end 299.706251 42.1) (width 0.45) (layer F.Cu) (net 100))
+  (segment (start 299.706251 42.1) (end 300.7 42.1) (width 0.45) (layer F.Cu) (net 100))
+  (segment (start 294.46875 44.51875) (end 296.8875 42.1) (width 0.45) (layer F.Cu) (net 100))
+  (segment (start 299.656251 61.1) (end 300.7 61.1) (width 0.45) (layer F.Cu) (net 100))
+  (segment (start 296.9375 61.1) (end 299.656251 61.1) (width 0.45) (layer F.Cu) (net 100))
+  (segment (start 294.46875 63.56875) (end 296.9375 61.1) (width 0.45) (layer F.Cu) (net 100))
+  (segment (start 296.8875 80.2) (end 299.706251 80.2) (width 0.45) (layer F.Cu) (net 100))
+  (segment (start 299.706251 80.2) (end 300.7 80.2) (width 0.45) (layer F.Cu) (net 100))
+  (segment (start 294.46875 82.61875) (end 296.8875 80.2) (width 0.45) (layer F.Cu) (net 100))
+  (segment (start -0.0375 23) (end 2.39375 20.56875) (width 0.45) (layer F.Cu) (net 100))
+  (segment (start -4.2 23) (end -0.0375 23) (width 0.45) (layer F.Cu) (net 100))
+  (segment (start -4.2 99.2) (end -4.2 23) (width 0.45) (layer F.Cu) (net 100))
+  (segment (start -0.0375 99.2) (end -4.2 99.2) (width 0.45) (layer F.Cu) (net 100))
+  (segment (start 2.39375 96.76875) (end -0.0375 99.2) (width 0.45) (layer F.Cu) (net 100))
+  (segment (start -3.243751 42) (end -4.2 42) (width 0.45) (layer F.Cu) (net 100))
+  (segment (start 0.0125 42) (end -3.243751 42) (width 0.45) (layer F.Cu) (net 100))
+  (segment (start 2.39375 39.61875) (end 0.0125 42) (width 0.45) (layer F.Cu) (net 100))
+  (segment (start -3.193751 61.1) (end -4.2 61.1) (width 0.45) (layer F.Cu) (net 100))
+  (segment (start -0.0375 61.1) (end -3.193751 61.1) (width 0.45) (layer F.Cu) (net 100))
+  (segment (start 2.39375 58.66875) (end -0.0375 61.1) (width 0.45) (layer F.Cu) (net 100))
+  (segment (start -3.243751 80.1) (end -4.2 80.1) (width 0.45) (layer F.Cu) (net 100))
+  (segment (start 0.0125 80.1) (end -3.243751 80.1) (width 0.45) (layer F.Cu) (net 100))
+  (segment (start 2.39375 77.71875) (end 0.0125 80.1) (width 0.45) (layer F.Cu) (net 100))
+  (segment (start 2.39375 94.6) (end 2.5375 94.45625) (width 0.45) (layer F.Cu) (net 100))
+  (segment (start 2.39375 96.76875) (end 2.39375 94.6) (width 0.45) (layer F.Cu) (net 100))
+  (segment (start 2.5375 20.425) (end 2.39375 20.56875) (width 0.45) (layer F.Cu) (net 100))
+  (segment (start 2.5375 18.25625) (end 2.5375 20.425) (width 0.45) (layer F.Cu) (net 100))
+  (segment (start 2.5375 39.475) (end 2.39375 39.61875) (width 0.45) (layer F.Cu) (net 100))
+  (segment (start 2.5375 37.30625) (end 2.5375 39.475) (width 0.45) (layer F.Cu) (net 100))
+  (segment (start 2.5375 58.525) (end 2.39375 58.66875) (width 0.45) (layer F.Cu) (net 100))
+  (segment (start 2.5375 56.35625) (end 2.5375 58.525) (width 0.45) (layer F.Cu) (net 100))
+  (segment (start 2.5375 77.575) (end 2.39375 77.71875) (width 0.45) (layer F.Cu) (net 100))
+  (segment (start 2.5375 75.40625) (end 2.5375 77.575) (width 0.45) (layer F.Cu) (net 100))
+  (segment (start 294.46875 31.252466) (end 294.46875 39.61875) (width 0.3) (layer F.Cu) (net 104))
+  (segment (start 297.66875 28.052466) (end 294.46875 31.252466) (width 0.3) (layer F.Cu) (net 104))
+  (segment (start 297.66875 25.46875) (end 297.66875 28.052466) (width 0.3) (layer F.Cu) (net 104))
+  (segment (start 294.46875 50.302466) (end 294.46875 58.66875) (width 0.3) (layer F.Cu) (net 105))
+  (segment (start 297.66875 47.102466) (end 294.46875 50.302466) (width 0.3) (layer F.Cu) (net 105))
+  (segment (start 297.66875 44.51875) (end 297.66875 47.102466) (width 0.3) (layer F.Cu) (net 105))
+  (segment (start 294.46875 69.352466) (end 294.46875 77.71875) (width 0.3) (layer F.Cu) (net 106))
+  (segment (start 297.66875 66.152466) (end 294.46875 69.352466) (width 0.3) (layer F.Cu) (net 106))
+  (segment (start 297.66875 63.56875) (end 297.66875 66.152466) (width 0.3) (layer F.Cu) (net 106))
+  (segment (start 297.66875 85.202466) (end 294.46875 88.402466) (width 0.3) (layer F.Cu) (net 107))
+  (segment (start 294.46875 88.402466) (end 294.46875 96.76875) (width 0.3) (layer F.Cu) (net 107))
+  (segment (start 297.66875 82.61875) (end 297.66875 85.202466) (width 0.3) (layer F.Cu) (net 107))
+  (segment (start 8.902751 108.177751) (end 2.39375 101.66875) (width 0.3) (layer F.Cu) (net 108))
+  (segment (start 293.743465 108.177751) (end 8.902751 108.177751) (width 0.3) (layer F.Cu) (net 108))
+  (segment (start 297.66875 104.252466) (end 293.743465 108.177751) (width 0.3) (layer F.Cu) (net 108))
+  (segment (start 297.66875 101.66875) (end 297.66875 104.252466) (width 0.3) (layer F.Cu) (net 108))
+  (segment (start 2.39375 90.985034) (end 2.39375 82.61875) (width 0.3) (layer F.Cu) (net 109))
+  (segment (start -0.80625 94.185034) (end 2.39375 90.985034) (width 0.3) (layer F.Cu) (net 109))
+  (segment (start -0.80625 96.76875) (end -0.80625 94.185034) (width 0.3) (layer F.Cu) (net 109))
+  (segment (start 2.39375 71.935034) (end 2.39375 63.56875) (width 0.3) (layer F.Cu) (net 110))
+  (segment (start -0.80625 75.135034) (end 2.39375 71.935034) (width 0.3) (layer F.Cu) (net 110))
+  (segment (start -0.80625 77.71875) (end -0.80625 75.135034) (width 0.3) (layer F.Cu) (net 110))
+  (segment (start 2.39375 52.885034) (end 2.39375 44.51875) (width 0.3) (layer F.Cu) (net 111))
+  (segment (start -0.80625 56.085034) (end 2.39375 52.885034) (width 0.3) (layer F.Cu) (net 111))
+  (segment (start -0.80625 58.66875) (end -0.80625 56.085034) (width 0.3) (layer F.Cu) (net 111))
+  (segment (start 2.39375 33.835034) (end 2.39375 25.46875) (width 0.3) (layer F.Cu) (net 112))
+  (segment (start -0.80625 37.035034) (end 2.39375 33.835034) (width 0.3) (layer F.Cu) (net 112))
+  (segment (start -0.80625 39.61875) (end -0.80625 37.035034) (width 0.3) (layer F.Cu) (net 112))
   (zone (net 90) (net_name GND) (layer F.Cu) (hatch edge 0.508)
     (connect_pads (clearance 0.508))

Commit message: finish routing
Parts:
- moved R2 3.97 mm to (30.2, 0.77)
- moved Q1 3.97 mm to (34.9, 0.79)
- moved R1 3.85 mm to (39.7, 0.94)
Connections:
- U1 pad 10: COL14 -> COL8
- U1 pad 11: COL13 -> COL9
- U1 pad 12: COL12 -> COL10
- U1 pad 14: COL10 -> COL12
- U1 pad 15: COL9 -> COL13
- U1 pad 16: COL8 -> COL14
- U1 pad 17: COL7 -> RGB
- U1 pad 7: RGB -> COL7
Routing:
- net +5V: track 251.6 -> 617.9 mm
- net COL14: track 88.0 -> 358.9 mm
- net RGB_DIN: track 0.00 -> 266.7 mm
- net COL13: track 108.6 -> 353.5 mm
- net COL12: track 103.5 -> 331.8 mm
- net COL11: track 103.5 -> 315.3 mm
- net COL10: track 103.5 -> 298.8 mm
- net COL9: track 103.5 -> 282.3 mm
- net COL8: track 103.5 -> 265.8 mm
- net COL7: track 107.4 -> 258.3 mm
- net COL6: track 115.0 -> 220.2 mm
- net ROW5: track 266.7 -> 371.3 mm
- net COL5: track 115.0 -> 203.5 mm
- net ROW4: track 257.2 -> 345.0 mm
- net COL4: track 115.0 -> 187.2 mm
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
Commit message: make all traces same size
Other:
- board outline added: 349.1 x 130.9 mm
- net class PWR removed

Commit message: add mounting holes and shift dev board
Parts:
- added H1: MountingHole_Pad, MountingHole:MountingHole_2.2mm_M2_Pad_TopBottom, F.Cu at (83.3, -27.8)
- added H2: MountingHole_Pad, MountingHole:MountingHole_2.2mm_M2_Pad_TopBottom, F.Cu at (83.3, -21.8)
- added H3: MountingHole_Pad, MountingHole:MountingHole_2.2mm_M2_Pad_TopBottom, F.Cu at (89.3, -27.8)
- added H4: MountingHole_Pad, MountingHole:MountingHole_2.2mm_M2_Pad_TopBottom, F.Cu at (89.3, -21.8)
- moved R1 12.7 mm to (52.4, 0.00)
- moved Q1 12.7 mm to (47.6, 0.00)
- moved R2 12.7 mm to (42.9, 0.00)
- moved U1 11.9 mm to (11.1, 3.17)
Routing:
- net RGB_DIN: track 266.7 -> 254.4 mm
- net COL3: track 170.7 -> 158.7 mm
- net COL4: track 187.2 -> 175.3 mm
- net COL11: track 315.3 -> 303.4 mm
- net COL8: track 265.8 -> 253.9 mm
- net COL7: track 258.3 -> 246.4 mm
- net COL9: track 282.3 -> 270.4 mm
- net COL6: track 220.2 -> 208.3 mm
- net COL2: track 154.1 -> 142.2 mm
- net COL14: track 358.9 -> 347.0 mm
- net COL13: track 353.5 -> 341.6 mm
- net COL12: track 331.8 -> 319.9 mm
- net COL10: track 298.8 -> 286.9 mm
- net COL1: track 114.6 -> 102.7 mm
- net COL5: track 203.5 -> 191.8 mm
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- added copper zone on B.Cu, net GND
