File: smol.kicad_pcb (KiCad board)
At the start: 2 copper layers, 349.1 x 130.9 mm, 168 parts, among them Q1 BSS138, SW1 1U, SW10 1U, SW11 1U, SW12 1U, SW13 1U, SW14 2U, SW15 2U, SW16 1U, SW17 1U, SW18 1U, SW19 1U, SW2 1U, SW20 1U, SW21 1U, SW22 1U, SW23 1U, SW24 1U, SW25 1U, SW26 1U, SW27 1U, SW28 1U, SW29 1U, SW3 1U, SW30 1U, SW31 1U, SW32 1U, SW33 1U, SW34 1U, SW35 1U, SW36 1U, SW37 1U, SW38 1U, SW39 1U, SW4 1U, SW40 1U, SW41 1U, SW42 2U, SW43 2U, SW44 1U, SW45 1U, SW46 1U, SW47 1U, SW48 1U, SW49 1U, SW5 1U, SW50 1U, SW51 1U, SW52 1U, SW53 1U, SW54 1U, SW55 1U, SW56 1U, SW57 1U, SW58 1U, SW59 1U, SW6 1U, SW60 1U, SW61 1U, SW62 1U, SW63 2U, SW64 1U, SW65 1U, SW66 1U, SW67 1U, SW68 1U, SW69 1U, SW7 1U, SW70 1U, SW8 1U, SW9 1U, U1 MiniF4x1Cx_V31

Commit message: finalize and prepare to export for order
Parts:
- added G***: LOGO, libraries:qr-code, B.Cu at (285.0, -0.79)
- added REF**: OSHW-Logo2_24.3x20mm_SilkScreen, Symbol:OSHW-Logo2_24.3x20mm_SilkScreen, F.Cu at (288.9, -2.00)
- moved H3 256.8 mm to (305.2, 111.3)
- moved H2 222.2 mm to (305.2, -9.80)
- moved H4 165.1 mm to (-8.27, 111.3)
- moved H1 93.4 mm to (-8.27, -9.80)
Routing:
- net +5V: track 608.2 -> 613.3 mm
- net Net-(RGB5-Pad4): track 302.2 -> 302.7 mm
Other:
- board size 349.1 x 130.9 mm -> 327.4 x 135.1 mm
- board text added: ""Pyrotelekinetic""
- board text added: "Smol V1.0 Carter Ison"
- board text added: "https://github.com/Pyrotelekinetic/smol"

Commit message: finalize aesthetics
Parts:
- removed the G*** at (285.0, -0.79)
- added G***: LOGO, libraries:bee, F.Cu at (138.9, 110.3)
- added G***: LOGO, libraries:SMOL, F.Cu at (138.9, -2.38)
- added G***: LOGO, libraries:qr-code-invert, B.Cu at (285.8, -1.50)
Other:
- board text added: ""apioform""
- board text added: "SMOL V1.0 Carter Ison"
- board text removed: "Smol V1.0 Carter Ison"
